Commit message: FT Compensation attempt

File: src/ur5_workbench_description/urdf/ur5_workbench.urdf.xacro (robot description, xacro)
@@ -24,5 +24,5 @@
     thing2_visual_parameters_file="$(arg thing2_visual_parameters_file)"
   >
-    <origin xyz="0 0 1" rpy="0 0 0" />
+    <origin xyz="0 0 0" rpy="0 0 0" />
   </xacro:ur5_workbench>
 </robot>

File: src/ur5_workbench_description/urdf/ur5_workbench_macro.xacro (robot description, xacro)
@@ -31,5 +31,5 @@
       <parent link="table" />
       <child link="thing1_robot_mount" />
-      <origin xyz="0.2 0.3 0" rpy="0 0 ${pi}" />
+      <origin xyz="0.381 0.381 0" rpy="0 0 ${pi}" />
     </joint>
     <xacro:ur_robot
@@ -44,6 +44,6 @@
       <origin xyz="0 0 0" rpy="0 0 0" />
     </xacro:ur_robot>
-    <xacro:robotiq_ft300 parent="flange" tf_prefix="thing1_">
-      <origin xyz="0 0 0" rpy="0 0 0" />
+    <xacro:robotiq_ft300 parent="tool0" tf_prefix="thing1_">
+      <origin xyz="0 0 -0.004" rpy="0 0 0" />
     </xacro:robotiq_ft300>
     <xacro:if value="${include_ros2_control}">
@@ -55,5 +55,5 @@
     <xacro:robotiq_gripper
       name="thing1_robotiq_gripper"
-      parent="thing1_ft300_sensor"
+      parent="thing1_robotiq_ft_frame_id"
       prefix="thing1_"
       include_ros2_control="${include_ros2_control}"
@@ -65,5 +65,5 @@
       <parent link="table" />
       <child link="thing2_robot_mount" />
-      <origin xyz="1.2 0.3 0" rpy="0 0 ${pi}" />
+      <origin xyz="1.905 0.381 0" rpy="0 0 ${pi}" />
     </joint>
     <xacro:ur_robot
@@ -78,6 +78,6 @@
       <origin xyz="0 0 0" rpy="0 0 0" />
     </xacro:ur_robot>
-    <xacro:robotiq_ft300 parent="flange" tf_prefix="thing2_">
-      <origin xyz="0 0 0" rpy="0 0 0" />
+    <xacro:robotiq_ft300 parent="tool0" tf_prefix="thing2_">
+      <origin xyz="0 0 -0.004" rpy="0 0 0" />
     </xacro:robotiq_ft300>
     <xacro:if value="${include_ros2_control}">
@@ -89,5 +89,5 @@
     <xacro:robotiq_gripper
       name="thing2_robotiq_gripper"
-      parent="thing2_ft300_sensor"
+      parent="thing2_robotiq_ft_frame_id"
       prefix="thing2_"
       include_ros2_control="${include_ros2_control}"

File: src/ur5_workbench_mujoco_config/urdf/ur5_workbench.mujoco_ros2_control.xacro (robot description, xacro)
@@ -58,7 +58,5 @@
       <state_interface name="velocity" />
       <state_interface name="effort" />
-      <control_interface name="position" />
-      <control_interface name="velocity" />
-      <control_interface name="effort" />
+      <command_interface name="position" />
     </joint>
   </xacro:macro>
@@ -80,7 +78,7 @@
       initial_position="0.0"
     />
-    <!-- <sensor name="${prefix}robotiq_ft_frame_id">
+    <sensor name="${prefix}tcp_fts_sensor">
       <param name="mujoco_type">fts</param>
-      <param name="mujoco_sensor_name">${prefix}robotiq_ft_frame_id</param>
+      <param name="mujoco_sensor_name">${prefix}tcp_fts_sensor</param>
       <state_interface name="force.x" />
       <state_interface name="force.y" />
@@ -89,12 +87,104 @@
       <state_interface name="torque.y" />
       <state_interface name="torque.z" />
-    </sensor> -->
+    </sensor>
   </xacro:macro>
+  <mujoco_inputs>
+    <raw_inputs>
+      <option integrator="implicitfast"/>
+      <default>
+        <material specular="0.5" shininess="0.25"/>
+        <joint axis="0 1 0" range="-6.28319 6.28319" armature="0.1"/>
+        <position ctrlrange="-6.2831 6.2831"/>
+        <general biastype="affine" ctrlrange="-6.2831 6.2831" />
+        <default class="size4">
+          <joint damping="10"/>
+          <general forcerange="-330 330" gainprm="100000" biasprm="0 -100000 -10000" />
+        </default>
+        <default class="size3">
+          <joint damping="5"/>
+          <general forcerange="-150 150" gainprm="40000" biasprm="0 -40000 -4000" />
+          <default class="size3_limited">
+            <joint range="-3.1415 3.1415"/>
+            <general ctrlrange="-3.1415 3.1415" />
+          </default>
+        </default>
+        <default class="size2">
+          <joint damping="2"/>
+          <general forcerange="-56 56" gainprm="10000" biasprm="0 -10000 -1000" />
+        </default>
+        <default class="visual">
+          <geom group="2" type="mesh" contype="0" conaffinity="0"/>
+        </default>
+        <default class="collision">
+          <geom group="3" type="mesh"/>
+        </default>
+      </default>
+      <actuator>
+        <position class="size4" name="thing1_shoulder_pan_joint" joint="thing1_shoulder_pan_joint"/>
+        <position class="size4" name="thing1_shoulder_lift_joint" joint="thing1_shoulder_lift_joint"/>
+        <position class="size3_limited" name="thing1_elbow_joint" joint="thing1_elbow_joint"/>
+        <position class="size2" name="thing1_wrist_1_joint" joint="thing1_wrist_1_joint"/>
+        <position class="size2" name="thing1_wrist_2_joint" joint="thing1_wrist_2_joint"/>
+        <position class="size2" name="thing1_wrist_3_joint" joint="thing1_wrist_3_joint"/>
+        <position class="size2" name="thing1_robotiq_85_left_knuckle_joint" joint="thing1_robotiq_85_left_knuckle_joint"/>
+        <position class="size4" name="thing2_shoulder_pan_joint" joint="thing2_shoulder_pan_joint"/>
+        <position class="size4" name="thing2_shoulder_lift_joint" joint="thing2_shoulder_lift_joint"/>
+        <position class="size3_limited" name="thing2_elbow_joint" joint="thing2_elbow_joint"/>
+        <position class="size2" name="thing2_wrist_1_joint" joint="thing2_wrist_1_joint"/>
+        <position class="size2" name="thing2_wrist_2_joint" joint="thing2_wrist_2_joint"/>
+        <position class="size2" name="thing2_wrist_3_joint" joint="thing2_wrist_3_joint"/>
+        <position class="size2" name="thing2_robotiq_85_left_knuckle_joint" joint="thing2_robotiq_85_left_knuckle_joint" />
+      </actuator>
+      <equality>
+        <joint joint1="thing1_robotiq_85_left_knuckle_joint" joint2="thing1_robotiq_85_right_knuckle_joint" polycoef="0 -1 0 0 0" solimp="0.95 0.99 0.001" solref="0.005 1"/>
+        <joint joint1="thing1_robotiq_85_left_knuckle_joint" joint2="thing1_robotiq_85_left_inner_knuckle_joint" polycoef="0 1 0 0 0" solimp="0.95 0.99 0.001" solref="0.005 1"/>
+        <joint joint1="thing1_robotiq_85_left_knuckle_joint" joint2="thing1_robotiq_85_right_inner_knuckle_joint" polycoef="0 -1 0 0 0" solimp="0.95 0.99 0.001" solref="0.005 1"/>
+        <joint joint1="thing1_robotiq_85_left_knuckle_joint" joint2="thing1_robotiq_85_left_finger_tip_joint" polycoef="0 -1 0 0 0" solimp="0.95 0.99 0.001" solref="0.005 1"/>
+        <joint joint1="thing1_robotiq_85_left_knuckle_joint" joint2="thing1_robotiq_85_right_finger_tip_joint" polycoef="0 1 0 0 0" solimp="0.95 0.99 0.001" solref="0.005 1"/>
+        <joint joint1="thing2_robotiq_85_left_knuckle_joint" joint2="thing2_robotiq_85_right_knuckle_joint" polycoef="0 -1 0 0 0" solimp="0.95 0.99 0.001" solref="0.005 1"/>
+        <joint joint1="thing2_robotiq_85_left_knuckle_joint" joint2="thing2_robotiq_85_left_inner_knuckle_joint" polycoef="0 1 0 0 0" solimp="0.95 0.99 0.001" solref="0.005 1"/>
+        <joint joint1="thing2_robotiq_85_left_knuckle_joint" joint2="thing2_robotiq_85_right_inner_knuckle_joint" polycoef="0 -1 0 0 0" solimp="0.95 0.99 0.001" solref="0.005 1"/>
+        <joint joint1="thing2_robotiq_85_left_knuckle_joint" joint2="thing2_robotiq_85_left_finger_tip_joint" polycoef="0 -1 0 0 0" solimp="0.95 0.99 0.001" solref="0.005 1"/>
+        <joint joint1="thing2_robotiq_85_left_knuckle_joint" joint2="thing2_robotiq_85_right_finger_tip_joint" polycoef="0 1 0 0 0" solimp="0.95 0.99 0.001" solref="0.005 1"/>
+      </equality>
+      <sensor>
+        <force name="thing1_tcp_fts_sensor_force" site="thing1_robotiq_ft_frame_id"/>
+        <torque name="thing1_tcp_fts_sensor_torque" site="thing1_robotiq_ft_frame_id"/>
+      </sensor>
+      <sensor>
+        <force name="thing2_tcp_fts_sensor_force" site="thing2_robotiq_ft_frame_id"/>
+        <torque name="thing2_tcp_fts_sensor_torque" site="thing2_robotiq_ft_frame_id"/>
+      </sensor>
+    </raw_inputs>
+    <!-- Process arguments for the URDF -->
+    <processed_inputs>
+      <!-- Add frictionloss and armature to fingers to help with backdriving -->
+      <!-- <modify_element type="joint" name="thing1_robotiq_85_left_knuckle_joint" armature="0.5" frictionloss="5.0" />
+      <modify_element type="joint" name="thing1_robotiq_85_right_knuckle_joint" armature="0.5" frictionloss="5.0" /> -->
+      <!-- Add frictionloss and armature to fingers to help with backdriving -->
+      <!-- <modify_element type="joint" name="thing2_robotiq_85_left_knuckle_joint" armature="0.5" frictionloss="5.0" />
+      <modify_element type="joint" name="thing2_robotiq_85_right_knuckle_joint" armature="0.5" frictionloss="5.0" /> -->
+    </processed_inputs>
+    <scene>
+      <statistic center="0.4 0 0.4" extent="1"/>
+      <visual>
+        <headlight diffuse="0.6 0.6 0.6" ambient="0.1 0.1 0.1" specular="0 0 0"/>
+        <rgba haze="0.15 0.25 0.35 1"/>
+        <global azimuth="120" elevation="-20"/>
+      </visual>
+      <asset>
+        <texture type="skybox" builtin="gradient" rgb1="0.3 0.5 0.7" rgb2="0 0 0" width="512" height="3072"/>
+        <texture type="2d" name="groundplane" builtin="checker" mark="edge" rgb1="0.2 0.3 0.4" rgb2="0.1 0.2 0.3"
+          markrgb="0.8 0.8 0.8" width="300" height="300"/>
+        <material name="groundplane" texture="groundplane" texuniform="true" texrepeat="5 5"/>
+      </asset>
+      <worldbody>
+        <light pos="0 0 1.5" dir="0 0 -1" directional="true"/>
+      </worldbody>
+    </scene>
+  </mujoco_inputs>
   <ros2_control name="MujocoSystem" type="system">
     <hardware>
       <plugin>mujoco_ros2_control/MujocoSystemInterface</plugin>
-      <param
-        name="mujoco_model"
-      >$(find ur5_workbench_mujoco_config)/description/scene.xml</param>
       <param name="sim_speed_factor">1.0</param>
     </hardware>

Commit message: Updates to description + initialization of deply package

File: src/ur5_workbench_description/urdf/ur5_workbench.urdf.xacro (robot description, xacro)
@@ -3,8 +3,12 @@
   <xacro:include filename="$(find ur5_workbench_description)/urdf/ur5_workbench_macro.xacro" />
   <xacro:arg name="include_ros2_control" default="true"/>
+  <xacro:arg name="include_thing1" default="true"/>
+  <xacro:arg name="include_thing2" default="true"/>
+  <xacro:arg name="thing1_wrist_camera_model" default=""/>
   <xacro:arg name="thing1_joint_limits_parameters_file" default="$(find ur_description)/config/ur5/joint_limits.yaml"/>
   <xacro:arg name="thing1_kinematics_parameters_file" default="$(find ur_description)/config/ur5/default_kinematics.yaml"/>
   <xacro:arg name="thing1_physical_parameters_file" default="$(find ur_description)/config/ur5/physical_parameters.yaml"/>
   <xacro:arg name="thing1_visual_parameters_file" default="$(find ur_description)/config/ur5/visual_parameters.yaml"/>
+  <xacro:arg name="thing2_wrist_camera_model" default=""/>
   <xacro:arg name="thing2_joint_limits_parameters_file" default="$(find ur_description)/config/ur5/joint_limits.yaml"/>
   <xacro:arg name="thing2_kinematics_parameters_file" default="$(find ur_description)/config/ur5/default_kinematics.yaml"/>
@@ -15,8 +19,12 @@
     parent="world"
     include_ros2_control="$(arg include_ros2_control)"
+    include_thing1="$(arg include_thing1)"
+    include_thing2="$(arg include_thing2)"
+    thing1_wrist_camera_model="$(arg thing1_wrist_camera_model)"
     thing1_joint_limits_parameters_file="$(arg thing1_joint_limits_parameters_file)"
     thing1_kinematics_parameters_file="$(arg thing1_kinematics_parameters_file)"
     thing1_physical_parameters_file="$(arg thing1_physical_parameters_file)"
     thing1_visual_parameters_file="$(arg thing1_visual_parameters_file)"
+    thing2_wrist_camera_model="$(arg thing2_wrist_camera_model)"
     thing2_joint_limits_parameters_file="$(arg thing2_joint_limits_parameters_file)"
     thing2_kinematics_parameters_file="$(arg thing2_kinematics_parameters_file)"

File: src/ur5_workbench_description/urdf/ur5_workbench_macro.xacro (robot description, xacro)
@@ -1,8 +1,5 @@
 <?xml version="1.0" ?>
 <robot xmlns:xacro="http://www.ros.org/wiki/xacro">
-  <xacro:include filename="$(find ur_description)/urdf/ur_macro.xacro" />
-  <xacro:include filename="$(find robotiq_ft_sensor_description)/urdf/robotiq_ft300.urdf.xacro" />
-  <xacro:include filename="$(find robotiq_description)/urdf/robotiq_2f_85_macro.urdf.xacro" />
-  <xacro:include filename="$(find robotiq_ft_sensor_description)/urdf/robotiq_fts.ros2_control.xacro" />
+  <xacro:include filename="$(find ur5_workbench_description)/urdf/thing_macro.xacro" />
   <xacro:macro
     name="ur5_workbench"
@@ -11,8 +8,12 @@
       *origin
       include_ros2_control:=true
+      include_thing1:=true
+      thing1_wrist_camera_model
       thing1_joint_limits_parameters_file
       thing1_kinematics_parameters_file
       thing1_physical_parameters_file
       thing1_visual_parameters_file
+      include_thing2:=true
+      thing2_wrist_camera_model
       thing2_joint_limits_parameters_file
       thing2_kinematics_parameters_file
@@ -21,5 +22,5 @@
       "
   >
-    <joint name="table_base_joint" type="fixed">
+    <joint name="table_joint" type="fixed">
       <xacro:insert_block name="origin" />
       <parent link="${parent}" />
@@ -27,72 +28,32 @@
     </joint>
     <link name="table" />
-    <link name="thing1_robot_mount" />
-    <joint name="thing1_robot_mount_joint" type="fixed">
-      <parent link="table" />
-      <child link="thing1_robot_mount" />
-      <origin xyz="0.381 0.381 0" rpy="0 0 ${pi}" />
-    </joint>
-    <xacro:ur_robot
-      name="thing1"
-      tf_prefix="thing1_"
-      parent="thing1_robot_mount"
-      joint_limits_parameters_file="${thing1_joint_limits_parameters_file}"
-      kinematics_parameters_file="${thing1_kinematics_parameters_file}"
-      physical_parameters_file="${thing1_physical_parameters_file}"
-      visual_parameters_file="${thing1_visual_parameters_file}"
-    >
-      <origin xyz="0 0 0" rpy="0 0 0" />
-    </xacro:ur_robot>
-    <xacro:robotiq_ft300 parent="tool0" tf_prefix="thing1_">
-      <origin xyz="0 0 -0.004" rpy="0 0 0" />
-    </xacro:robotiq_ft300>
-    <xacro:if value="${include_ros2_control}">
-      <xacro:robotiq_fts_ros2_control
-        name="thing1_"
-        tf_prefix="thing1_"
-      />
+    <xacro:if value="${include_thing1}">
+      <xacro:thing
+        name="thing1"
+        parent="table"
+        include_ros2_control="${include_ros2_control}"
+        wrist_camera_model="${thing1_wrist_camera_model}"
+        joint_limits_parameters_file="${thing1_joint_limits_parameters_file}"
+        kinematics_parameters_file="${thing1_kinematics_parameters_file}"
+        physical_parameters_file="${thing1_physical_parameters_file}"
+        visual_parameters_file="${thing1_visual_parameters_file}"
+      >
+        <origin xyz="0.381 0.381 0" rpy="0 0 ${pi}" />
+      </xacro:thing>
     </xacro:if>
-    <xacro:robotiq_gripper
-      name="thing1_robotiq_gripper"
-      parent="thing1_robotiq_ft_frame_id"
-      prefix="thing1_"
-      include_ros2_control="${include_ros2_control}"
-    >
-      <origin xyz="0 0 0" rpy="0 0 0" />
-    </xacro:robotiq_gripper>
-    <link name="thing2_robot_mount" />
-    <joint name="thing2_robot_mount_joint" type="fixed">
-      <parent link="table" />
-      <child link="thing2_robot_mount" />
-      <origin xyz="1.905 0.381 0" rpy="0 0 ${pi}" />
-    </joint>
-    <xacro:ur_robot
-      name="thing2"
-      tf_prefix="thing2_"
-      parent="thing2_robot_mount"
-      joint_limits_parameters_file="${thing2_joint_limits_parameters_file}"
-      kinematics_parameters_file="${thing2_kinematics_parameters_file}"
-      physical_parameters_file="${thing2_physical_parameters_file}"
-      visual_parameters_file="${thing2_visual_parameters_file}"
-    >
-      <origin xyz="0 0 0" rpy="0 0 0" />
-    </xacro:ur_robot>
-    <xacro:robotiq_ft300 parent="tool0" tf_prefix="thing2_">
-      <origin xyz="0 0 -0.004" rpy="0 0 0" />
-    </xacro:robotiq_ft300>
-    <xacro:if value="${include_ros2_control}">
-      <xacro:robotiq_fts_ros2_control
-        name="thing2_"
-        tf_prefix="thing2_"
-      />
+    <xacro:if value="${include_thing2}">
+      <xacro:thing
+        name="thing2"
+        parent="table"
+        include_ros2_control="${include_ros2_control}"
+        wrist_camera_model="${thing2_wrist_camera_model}"
+        joint_limits_parameters_file="${thing2_joint_limits_parameters_file}"
+        kinematics_parameters_file="${thing2_kinematics_parameters_file}"
+        physical_parameters_file="${thing2_physical_parameters_file}"
+        visual_parameters_file="${thing2_visual_parameters_file}"
+      >
+        <origin xyz="1.905 0.381 0" rpy="0 0 ${pi}" />
+      </xacro:thing>
     </xacro:if>
-    <xacro:robotiq_gripper
-      name="thing2_robotiq_gripper"
-      parent="thing2_robotiq_ft_frame_id"
-      prefix="thing2_"
-      include_ros2_control="${include_ros2_control}"
-    >
-      <origin xyz="0 0 0" rpy="0 0 0" />
-    </xacro:robotiq_gripper>
   </xacro:macro>
 </robot>
