Commit message: Saved mjcf to mjcf_data, urdf configurable via xacro, initial ros2_control and moveit packages.

File: src/ur5_workbench_description/urdf/camera_mount_macro.xacro (robot description, xacro)
@@ -39,5 +39,5 @@
     </link>
     <joint name="${tf_prefix}tool_link_frame" type="fixed">
-      <origin xyz="0 0 0.00699997" rpy="0 0 0"/>
+      <origin xyz="0 0 0.00299997" rpy="0 0 0"/>
       <parent link="${tf_prefix}camera_mount_link"/>
       <child link="${tf_prefix}tool_link"/>

File: src/ur5_workbench_description/urdf/thing_macro.xacro (robot description, xacro)
@@ -29,5 +29,5 @@
     </xacro:ur_robot>
     <xacro:robotiq_ft300 parent="tool0" tf_prefix="${name}_">
-      <origin xyz="0 0 -0.004" rpy="0 0 0" />
+      <origin xyz="0 0 -0.004" rpy="0 0 ${-pi/2}" />
     </xacro:robotiq_ft300>
     <xacro:if value="${include_ros2_control}">

File: src/ur5_workbench_description/urdf/ur5_workbench_macro.xacro (robot description, xacro)
@@ -9,5 +9,5 @@
       include_ros2_control:=true
       include_thing1:=true
-      thing1_wrist_camera_model
+      thing1_wrist_camera_model:=''
       thing1_joint_limits_parameters_file
       thing1_kinematics_parameters_file
@@ -15,5 +15,5 @@
       thing1_visual_parameters_file
       include_thing2:=true
-      thing2_wrist_camera_model
+      thing2_wrist_camera_model:=''
       thing2_joint_limits_parameters_file
       thing2_kinematics_parameters_file
@@ -39,5 +39,5 @@
         visual_parameters_file="${thing1_visual_parameters_file}"
       >
-        <origin xyz="0.381 0.381 0" rpy="0 0 ${pi}" />
+        <origin xyz="1.905 0.381 0" rpy="0 0 ${pi/2}" />
       </xacro:thing>
     </xacro:if>
@@ -53,5 +53,5 @@
         visual_parameters_file="${thing2_visual_parameters_file}"
       >
-        <origin xyz="1.905 0.381 0" rpy="0 0 ${pi}" />
+        <origin xyz="0.381 0.381 0" rpy="0 0 ${pi/2}" />
       </xacro:thing>
     </xacro:if>

File: src/ur5_workbench_mujoco_config/urdf/ur5_workbench.mujoco_ros2_control.xacro (robot description, xacro)
@@ -54,5 +54,5 @@
     <joint name="${name}">
       <state_interface name="position">
-        <param name="initial_position">${initial_position}</param>
+        <param name="initial_value">${initial_position}</param>
       </state_interface>
       <state_interface name="velocity" />
@@ -68,8 +68,8 @@
     <xacro:mujoco_joint
       name="${prefix}shoulder_lift_joint"
-      initial_position="0.0"
+      initial_position="${-pi/2}"
     />
     <xacro:mujoco_joint name="${prefix}elbow_joint" initial_position="0.0" />
-    <xacro:mujoco_joint name="${prefix}wrist_1_joint" initial_position="0.0" />
+    <xacro:mujoco_joint name="${prefix}wrist_1_joint" initial_position="${-pi/2}" />
     <xacro:mujoco_joint name="${prefix}wrist_2_joint" initial_position="0.0" />
     <xacro:mujoco_joint name="${prefix}wrist_3_joint" initial_position="0.0" />
@@ -166,21 +166,4 @@
       <modify_element type="joint" name="thing2_robotiq_85_right_knuckle_joint" armature="0.5" frictionloss="5.0" /> -->
     </processed_inputs>
-    <scene>
-      <statistic center="0.4 0 0.4" extent="1"/>
-      <visual>
-        <headlight diffuse="0.6 0.6 0.6" ambient="0.1 0.1 0.1" specular="0 0 0"/>
-        <rgba haze="0.15 0.25 0.35 1"/>
-        <global azimuth="120" elevation="-20"/>
-      </visual>
-      <asset>
-        <texture type="skybox" builtin="gradient" rgb1="0.3 0.5 0.7" rgb2="0 0 0" width="512" height="3072"/>
-        <texture type="2d" name="groundplane" builtin="checker" mark="edge" rgb1="0.2 0.3 0.4" rgb2="0.1 0.2 0.3"
-          markrgb="0.8 0.8 0.8" width="300" height="300"/>
-        <material name="groundplane" texture="groundplane" texuniform="true" texrepeat="5 5"/>
-      </asset>
-      <worldbody>
-        <light pos="0 0 1.5" dir="0 0 -1" directional="true"/>
-      </worldbody>
-    </scene>
   </mujoco_inputs>
   <ros2_control name="MujocoSystem" type="system">
