Commit message: Stuff

File: mjcf_data/robot_description_formatted.urdf (robot description, URDF)
Before this commit: robot ur5_workbench, 52 links, 51 joints
Links:
- added link thing2_camera_link, mass 1e-9
- added link thing2_camera_mount_link, mass 1e-09; visual mesh filename=full/camera_mount.stl
- added link thing2_d405_bottom_screw_frame
- added link thing2_d405_link, mass 0.072; visual mesh filename=full/d405.stl scale=0.001 0.001 0.001
- added link thing2_tool_link, mass 1e-9
- added link thing2_wrist_camera_frame
Joints:
- added joint thing2_camera_link_frame: type fixed, parent thing2_camera_mount_link, child thing2_camera_link, origin xyz=-8.05759e-05 -0.0777769 0.00836815 rpy=-0.139625 3.04604e-07 -4.28088e-08, axis 0 0 0
- added joint thing2_camera_mount_joint: type fixed, parent thing2_robotiq_ft_frame_id, child thing2_camera_mount_link, origin xyz=0 0 0 rpy=0 0 0
- added joint thing2_d405_joint: type fixed, parent thing2_camera_link, child thing2_d405_bottom_screw_frame, origin xyz=0 0.021 0.009 rpy=0 -1.5707963267948966 1.5707963267948966
- added joint thing2_d405_link_joint: type fixed, parent thing2_d405_bottom_screw_frame, child thing2_d405_link, origin xyz=0.01085 0.009 0.021 rpy=0 0 0
- added joint thing2_tool_link_frame: type fixed, parent thing2_camera_mount_link, child thing2_tool_link, origin xyz=0 0 0.00299997 rpy=0 0 0, axis 0 0 0
- added joint thing2_wrist_camera_frame_joint: type fixed, parent thing2_d405_link, child thing2_wrist_camera_frame, origin xyz=0 0 0 rpy=-1.5707963267948966 0 -1.5707963267948966
- joint thing2_robotiq_85_base_joint: parent thing2_robotiq_ft_frame_id -> thing2_tool_link

File: src/ur5_workbench_mujoco_config/urdf/ur5_workbench.mujoco_ros2_control.xacro (robot description, xacro)
@@ -2,63 +2,59 @@
 <robot name="ur5_workbench" xmlns:xacro="http://www.ros.org/wiki/xacro">
   <xacro:include
-    filename="$(find ur5_workbench_description)/urdf/ur5_workbench_macro.xacro"
-  />
+        filename="$(find ur5_workbench_description)/urdf/ur5_workbench_macro.xacro"
+    />
   <xacro:arg name="include_thing1" default="true" />
   <xacro:arg name="include_thing2" default="true" />
-  <xacro:arg
-    name="thing1_wrist_camera_model"
-    default="" />
-  <xacro:arg
-    name="thing1_joint_limits_parameters_file"
-    default="$(find ur_description)/config/ur5/joint_limits.yaml"
-  />
-  <xacro:arg
-    name="thing1_kinematics_parameters_file"
-    default="$(find ur_description)/config/ur5/default_kinematics.yaml"
-  />
-  <xacro:arg
-    name="thing1_physical_parameters_file"
-    default="$(find ur_description)/config/ur5/physical_parameters.yaml"
-  />
-  <xacro:arg
-    name="thing1_visual_parameters_file"
-    default="$(find ur_description)/config/ur5/visual_parameters.yaml"
-  />
-  <xacro:arg
-    name="thing2_wrist_camera_model"
-    default="" />
-  <xacro:arg
-    name="thing2_joint_limits_parameters_file"
-    default="$(find ur_description)/config/ur5/joint_limits.yaml"
-  />
-  <xacro:arg
-    name="thing2_kinematics_parameters_file"
-    default="$(find ur_description)/config/ur5/default_kinematics.yaml"
-  />
-  <xacro:arg
-    name="thing2_physical_parameters_file"
-    default="$(find ur_description)/config/ur5/physical_parameters.yaml"
-  />
-  <xacro:arg
-    name="thing2_visual_parameters_file"
-    default="$(find ur_description)/config/ur5/visual_parameters.yaml"
-  />
+  <xacro:arg name="thing1_wrist_camera_model" default="" />
+  <xacro:arg
+        name="thing1_joint_limits_parameters_file"
+        default="$(find ur_description)/config/ur5/joint_limits.yaml"
+    />
+  <xacro:arg
+        name="thing1_kinematics_parameters_file"
+        default="$(find ur_description)/config/ur5/default_kinematics.yaml"
+    />
+  <xacro:arg
+        name="thing1_physical_parameters_file"
+        default="$(find ur_description)/config/ur5/physical_parameters.yaml"
+    />
+  <xacro:arg
+        name="thing1_visual_parameters_file"
+        default="$(find ur_description)/config/ur5/visual_parameters.yaml"
+    />
+  <xacro:arg name="thing2_wrist_camera_model" default="" />
+  <xacro:arg
+        name="thing2_joint_limits_parameters_file"
+        default="$(find ur_description)/config/ur5/joint_limits.yaml"
+    />
+  <xacro:arg
+        name="thing2_kinematics_parameters_file"
+        default="$(find ur_description)/config/ur5/default_kinematics.yaml"
+    />
+  <xacro:arg
+        name="thing2_physical_parameters_file"
+        default="$(find ur_description)/config/ur5/physical_parameters.yaml"
+    />
+  <xacro:arg
+        name="thing2_visual_parameters_file"
+        default="$(find ur_description)/config/ur5/visual_parameters.yaml"
+    />
   <link name="world" />
   <xacro:ur5_workbench
-    parent="world"
-    include_ros2_control="false"
-    include_thing1="$(arg include_thing1)"
-    include_thing2="$(arg include_thing2)"
-    thing1_wrist_camera_model="$(arg thing1_wrist_camera_model)"
-    thing1_joint_limits_parameters_file="$(arg thing1_joint_limits_parameters_file)"
-    thing1_kinematics_parameters_file="$(arg thing1_kinematics_parameters_file)"
-    thing1_physical_parameters_file="$(arg thing1_physical_parameters_file)"
-    thing1_visual_parameters_file="$(arg thing1_visual_parameters_file)"
-    thing2_wrist_camera_model="$(arg thing2_wrist_camera_model)"
-    thing2_joint_limits_parameters_file="$(arg thing2_joint_limits_parameters_file)"
-    thing2_kinematics_parameters_file="$(arg thing2_kinematics_parameters_file)"
-    thing2_physical_parameters_file="$(arg thing2_physical_parameters_file)"
-    thing2_visual_parameters_file="$(arg thing2_visual_parameters_file)"
-  >
+        parent="world"
+        include_ros2_control="false"
+        include_thing1="$(arg include_thing1)"
+        include_thing2="$(arg include_thing2)"
+        thing1_wrist_camera_model="$(arg thing1_wrist_camera_model)"
+        thing1_joint_limits_parameters_file="$(arg thing1_joint_limits_parameters_file)"
+        thing1_kinematics_parameters_file="$(arg thing1_kinematics_parameters_file)"
+        thing1_physical_parameters_file="$(arg thing1_physical_parameters_file)"
+        thing1_visual_parameters_file="$(arg thing1_visual_parameters_file)"
+        thing2_wrist_camera_model="$(arg thing2_wrist_camera_model)"
+        thing2_joint_limits_parameters_file="$(arg thing2_joint_limits_parameters_file)"
+        thing2_kinematics_parameters_file="$(arg thing2_kinematics_parameters_file)"
+        thing2_physical_parameters_file="$(arg thing2_physical_parameters_file)"
+        thing2_visual_parameters_file="$(arg thing2_visual_parameters_file)"
+    >
     <origin xyz="0 0 0" rpy="0 0 0" />
   </xacro:ur5_workbench>
@@ -75,22 +71,22 @@
   <xacro:macro name="mujoco_ur5" params="prefix">
     <xacro:mujoco_joint
-      name="${prefix}shoulder_pan_joint"
-      initial_position="0.0"
-    />
+            name="${prefix}shoulder_pan_joint"
+            initial_position="0.0"
+        />
     <xacro:mujoco_joint
-      name="${prefix}shoulder_lift_joint"
-      initial_position="${-pi/2}"
-    />
+            name="${prefix}shoulder_lift_joint"
+            initial_position="${-pi/2}"
+        />
     <xacro:mujoco_joint name="${prefix}elbow_joint" initial_position="0.0" />
     <xacro:mujoco_joint
-      name="${prefix}wrist_1_joint"
-      initial_position="${-pi/2}"
-    />
+            name="${prefix}wrist_1_joint"
+            initial_position="${-pi/2}"
+        />
     <xacro:mujoco_joint name="${prefix}wrist_2_joint" initial_position="0.0" />
     <xacro:mujoco_joint name="${prefix}wrist_3_joint" initial_position="0.0" />
     <xacro:mujoco_joint
-      name="${prefix}robotiq_85_left_knuckle_joint"
-      initial_position="0.0"
-    />
+            name="${prefix}robotiq_85_left_knuckle_joint"
+            initial_position="0.0"
+        />
     <sensor name="${prefix}tcp_fts_sensor">
       <param name="mujoco_type">fts</param>
@@ -108,4 +104,5 @@
       <option integrator="implicitfast" />
       <default>
+        <site rgba="0 0 0 0" />
         <material specular="0.5" shininess="0.25" />
         <joint axis="0 1 0" range="-6.28319 6.28319" armature="0.1" />
@@ -115,16 +112,16 @@
           <joint damping="10" />
           <general
-            forcerange="-330 330"
-            gainprm="100000"
-            biasprm="0 -100000 -10000"
-          />
+                        forcerange="-330 330"
+                        gainprm="100000"
+                        biasprm="0 -100000 -10000"
+                    />
         </default>
         <default class="size3">
           <joint damping="5" />
           <general
-            forcerange="-150 150"
-            gainprm="40000"
-            biasprm="0 -40000 -4000"
-          />
+                        forcerange="-150 150"
+                        gainprm="40000"
+                        biasprm="0 -40000 -4000"
+                    />
           <default class="size3_limited">
             <joint range="-3.1415 3.1415" />
@@ -135,8 +132,8 @@
           <joint damping="2" />
           <general
-            forcerange="-56 56"
-            gainprm="10000"
-            biasprm="0 -10000 -1000"
-          />
+                        forcerange="-56 56"
+                        gainprm="10000"
+                        biasprm="0 -10000 -1000"
+                    />
         </default>
         <default class="visual">
@@ -150,67 +147,81 @@
       <xacro:if value="$(arg include_thing1)">
         <position
-          class="size4"
-          name="thing1_shoulder_pan_joint"
-          joint="thing1_shoulder_pan_joint"
-        />
-        <position
-          class="size4"
-          name="thing1_shoulder_lift_joint"
-          joint="thing1_shoulder_lift_joint"
-        />
-        <position
-          class="size3_limited"
-          name="thing1_elbow_joint"
-          joint="thing1_elbow_joint"
-        />
-        <position
-          class="size2"
-          name="thing1_wrist_1_joint"
-          joint="thing1_wrist_1_joint"
-        />
-        <position
-          class="size2"
-          name="thing1_wrist_2_joint"
-          joint="thing1_wrist_2_joint"
-        />
-        <position
-          class="size2"
-          name="thing1_wrist_3_joint"
-          joint="thing1_wrist_3_joint"
-        />
-        <position tendon="thing1_split" name="thing1_robotiq_85_left_knuckle_joint" kp="10000" dampratio="1.0" ctrlrange="0.0 0.79" forcerange="-150 150"/>
+                        class="size4"
+                        name="thing1_shoulder_pan_joint"
+                        joint="thing1_shoulder_pan_joint"
+                    />
+        <position
+                        class="size4"
+                        name="thing1_shoulder_lift_joint"
+                        joint="thing1_shoulder_lift_joint"
+                    />
+        <position
+                        class="size3_limited"
+                        name="thing1_elbow_joint"
+                        joint="thing1_elbow_joint"
+                    />
+        <position
+                        class="size2"
+                        name="thing1_wrist_1_joint"
+                        joint="thing1_wrist_1_joint"
+                    />
+        <position
+                        class="size2"
+                        name="thing1_wrist_2_joint"
+                        joint="thing1_wrist_2_joint"
+                    />
+        <position
+                        class="size2"
+                        name="thing1_wrist_3_joint"
+                        joint="thing1_wrist_3_joint"
+                    />
+        <position
+                        tendon="thing1_split"
+                        name="thing1_robotiq_85_left_knuckle_joint"
+                        kp="10000"
+                        dampratio="1.0"
+                        ctrlrange="0.0 0.79"
+                        forcerange="-150 150"
+                    />
       </xacro:if>
       <xacro:if value="$(arg include_thing2)">
         <position
-          class="size4"
-          name="thing2_shoulder_pan_joint"
-          joint="thing2_shoulder_pan_joint"
-        />
-        <position
-          class="size4"
-          name="thing2_shoulder_lift_joint"
-          joint="thing2_shoulder_lift_joint"
-        />
-        <position
-          class="size3_limited"
-          name="thing2_elbow_joint"
-          joint="thing2_elbow_joint"
-        />
-        <position
-          class="size2"
-          name="thing2_wrist_1_joint"
-          joint="thing2_wrist_1_joint"
-        />
-        <position
-          class="size2"
-          name="thing2_wrist_2_joint"
-          joint="thing2_wrist_2_joint"
-        />
-        <position
-          class="size2"
-          name="thing2_wrist_3_joint"
-          joint="thing2_wrist_3_joint"
-        />
-        <position tendon="thing2_split" name="thing2_robotiq_85_left_knuckle_joint" kp="10000" dampratio="1.0" ctrlrange="0.0 0.79" forcerange="-150 150"/>
+                        class="size4"
+                        name="thing2_shoulder_pan_joint"
+                        joint="thing2_shoulder_pan_joint"
+                    />
+        <position
+                        class="size4"
+                        name="thing2_shoulder_lift_joint"
+                        joint="thing2_shoulder_lift_joint"
+                    />
+        <position
+                        class="size3_limited"
+                        name="thing2_elbow_joint"
+                        joint="thing2_elbow_joint"
+                    />
+        <position
+                        class="size2"
+                        name="thing2_wrist_1_joint"
+                        joint="thing2_wrist_1_joint"
+                    />
+        <position
+                        class="size2"
+                        name="thing2_wrist_2_joint"
+                        joint="thing2_wrist_2_joint"
+                    />
+        <position
+                        class="size2"
+                        name="thing2_wrist_3_joint"
+                        joint="thing2_wrist_3_joint"
+                    />
+        <position
+                        tendon="thing2_split"
+                        name="thing2_robotiq_85_left_knuckle_joint"
+                        kp="10000"
+                        dampratio="1.0"
+                        ctrlrange="0.0 0.79"
+                        forcerange="-150 150"
+                    />
         </xacro:if>
       </actuator>
@@ -218,12 +229,12 @@
         <xacro:if value="$(arg include_thing1)">
         <fixed name="thing1_split">
-          <joint joint="thing1_robotiq_85_left_knuckle_joint" coef="0.5"/>
-          <joint joint="thing1_robotiq_85_right_knuckle_joint" coef="-0.5"/>
+          <joint joint="thing1_robotiq_85_left_knuckle_joint" coef="0.5" />
+          <joint joint="thing1_robotiq_85_right_knuckle_joint" coef="-0.5" />
         </fixed>
         </xacro:if>
         <xacro:if value="$(arg include_thing2)">
         <fixed name="thing2_split">
-          <joint joint="thing2_robotiq_85_left_knuckle_joint" coef="0.5"/>
-          <joint joint="thing2_robotiq_85_right_knuckle_joint" coef="-0.5"/>
+          <joint joint="thing2_robotiq_85_left_knuckle_joint" coef="0.5" />
+          <joint joint="thing2_robotiq_85_right_knuckle_joint" coef="-0.5" />
         </fixed>
         </xacro:if>
@@ -233,125 +244,199 @@
         <exclude body1="world" body2="thing1_shoulder_link" />
         <exclude
-          body1="thing1_wrist_3_link"
-          body2="thing1_robotiq_85_left_knuckle_link"
-        />
-        <exclude
-          body1="thing1_wrist_3_link"
-          body2="thing1_robotiq_85_left_inner_knuckle_link"
-        />
-        <exclude
-          body1="thing1_robotiq_85_left_inner_knuckle_link"
-          body2="thing1_robotiq_85_left_finger_tip_link"
-        />
-        <exclude
-          body1="thing1_robotiq_85_left_knuckle_link"
-          body2="thing1_robotiq_85_left_finger_tip_link"
-        />
-        <exclude
-          body1="thing1_wrist_3_link"
-          body2="thing1_robotiq_85_right_knuckle_link"
-        />
-        <exclude
-          body1="thing1_wrist_3_link"
-          body2="thing1_robotiq_85_right_inner_knuckle_link"
-        />
-        <exclude
-          body1="thing1_robotiq_85_right_inner_knuckle_link"
-          body2="thing1_robotiq_85_right_finger_tip_link"
-        />
-        <exclude
-          body1="thing1_robotiq_85_right_knuckle_link"
-          body2="thing1_robotiq_85_right_finger_tip_link"
-        />
-        <exclude body1="thing1_robotiq_85_left_finger_tip_link" body2="thing1_robotiq_85_right_finger_tip_link" />
-        </xacro:if>
-        <xacro:if value="$(arg include_thing2)" >
+                        body1="thing1_wrist_3_link"
+                        body2="thing1_robotiq_85_left_knuckle_link"
+                    />
+        <exclude
+                        body1="thing1_wrist_3_link"
+                        body2="thing1_robotiq_85_left_inner_knuckle_link"
+                    />
+        <exclude
+                        body1="thing1_robotiq_85_left_inner_knuckle_link"
+                        body2="thing1_robotiq_85_left_finger_tip_link"
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